File: tec_controller/tec_controller_v3.brd (EAGLE design)
At the start: 80 x 60 mm, 24 parts, among them IC1 LM358N, Q1 IRF512, Q2 IRF512

Commit message: adjustments to tec controller board and schematic
Parts:
- R4, R5: value (none) -> 1.3k
Changed lines of the file:
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@@
 <element name="PUMP1" library="SparkFun-Connectors" package="1X02_LOCK_LONGPADS" value="M02LOCK_LONGPADS" x="39.5" y="56" smashed="yes" rot="R180"/>
 <element name="CONTROL" library="SparkFun-Connectors" package="MOLEX-1X4" value="" x="56" y="56"/>
-<element name="R4" library="rcl" package="M0805" value="" x="30" y="21.5" smashed="yes" rot="MR180">
+<element name="R4" library="rcl" package="M0805" value="1.3k" x="30" y="21.5" smashed="yes" rot="MR180">
 <attribute name="NAME" x="28.73" y="20.23" size="1.27" layer="26" rot="MR180"/>
 <attribute name="VALUE" x="28.73" y="24.04" size="1.27" layer="28" rot="MR180"/>
 </element>
-<element name="R5" library="rcl" package="M0805" value="" x="50.5" y="21.5" rot="MR0"/>
+<element name="R5" library="rcl" package="M0805" value="1.3k" x="50.5" y="21.5" rot="MR0"/>
 <element name="IC1" library="linear" package="DIL08" value="LM358N" x="40" y="30" rot="R270"/>
 <element name="C5" library="rcl" package="C0805" value="100n" x="40" y="37" rot="MR0"/>
